File: docs/hardware/kicad/wheel_harness.kicad_sch (KiCad schematic)
At the start: 38 parts, among them SW1 battery master, U1 TCA9548A 0x70, U2 TCA9548A 0x71, U3 IMU module

Commit message: Hardware: KiCad ERC clean, netlist cross-check passes, SPICE results recorded
ERC 0 errors / 0 warnings; the netlist KiCad extracts matches harness_spec.py
on all 45 nets; BOM matches the drawing's parts list. ngspice confirms
152.8 ns rise at 2.2 k (pass) and 326.5 ns at 4.7 k (fail), and 4.97 V at the
worst pad on the 5 V ring.
Connections:
- net +12V_ESP: now also PWR3.1 (pwr)
- net +12V_PI: now also PWR2.1 (pwr)
- net +3V3: now also A1.3 (3V3); no longer PWR3.1 (pwr)
- net +5V_ESP: now also A1.1 (VBUS_USB)
- net +5V_PAD: now also A1.6 (5V); no longer PWR2.1 (pwr)
- net GND: now also A1.2 (GND)
- net SCL_MAIN: now also A1.5 (IO22_SCL)
- net SDA_MAIN: now also A1.4 (IO21_SDA)
